Commit message: Nav2 odometry smoothin ekf set up and working. Needs tuning

File: description/lidar.xacro (robot description, xacro)
@@ -16,5 +16,5 @@
         <collision>
             <geometry>
-                <cylinder radius="0.05" length="0.04"/>
+                <cylinder radius="0.05" length="0.05"/>
             </geometry>
         </collision>

File: description/robot.urdf.xacro (robot description, xacro)
@@ -6,3 +6,5 @@
     <xacro:include filename="lidar.xacro" />
     <xacro:include filename="camera.xacro" />
+    <xacro:include filename="imu.xacro" />
+    <!--<xacro:include filename="contact_switch.xacro" /> -->
 </robot>

File: description/robot_core.xacro (robot description, xacro)
@@ -26,5 +26,5 @@
         <parent link="base_link"/>
         <child link="base_footprint"/>
-        <origin xyz="0 0 0" rpy="0 0 0"/>
+        <origin xyz="0 0 -${wheel_radius}" rpy="0 0 0"/>
     </joint>
     <link name="base_footprint">
@@ -34,5 +34,5 @@
         <parent link="base_link"/>
         <child link="chassis"/>
-        <origin xyz="-${wheel_radius} 0 ${wheel_radius}"/>
+        <origin xyz="-${wheel_radius} 0 0"/>
     </joint>
     <link name="chassis">
@@ -58,5 +58,5 @@
         <parent link="base_link"/>
         <child link="left_wheel"/>
-        <origin xyz="0 ${wheel_offset} ${wheel_radius}" rpy="-${pi/2} 0 0"/>
+        <origin xyz="0 ${wheel_offset} 0" rpy="-${pi/2} 0 0"/>
         <axis xyz="0 0 1"/>
         <limit effort="${wheel_torque}" velocity="${wheel_speed}"/>
@@ -87,5 +87,5 @@
         <parent link="base_link"/>
         <child link="right_wheel"/>
-        <origin xyz="0 -${wheel_offset} ${wheel_radius}" rpy="${pi/2} 0 0"/>
+        <origin xyz="0 -${wheel_offset} 0" rpy="${pi/2} 0 0"/>
         <axis xyz="0 0 -1"/>
         <limit effort="${wheel_torque}" velocity="${wheel_speed}"/>

File: description/ros2_control.xacro (robot description, xacro)
@@ -41,11 +41,13 @@
         </plugin>
         <plugin
-            filename="gz-sim-user-commands-system"
-            name="gz::sim::systems::UserCommands">
+            filename="gz-sim-imu-system"
+            name="gz::sim::systems::Imu">
         </plugin>
+        <!--
         <plugin
-            filename="gz-sim-scene-broadcaster-system"
-            name="gz::sim::systems::SceneBroadcaster">
+            filename="gz-sim-contact-system"
+            name="gz::sim::systems::Contact">
         </plugin>
+         -->
     </gazebo>
 </robot>
