Commit message: cleaned up file(s)/structure a bit

File: description/XXXgazebo_control.xacro (robot description, xacro)
@@ -1,4 +1,8 @@
 <?xml version="1.0"?>
 <robot xmlns:xacro="http://www.ros.org/wiki/xacro">
+<!--OBSOLETE AND UNUSED-->
+<!--Introduced at the beginning of the Articulated Robotics tutorials,
+but then phased out in favor of ros2_control.xacro-->
+<!--Plug-ins for simulating various aspects of the robot in Gazebo-->
     <gazebo>
         <plugin name="gz::sim::systems::DiffDrive" filename="gz-sim-diff-drive-system">

File: description/camera.xacro (robot description, xacro)
@@ -1,4 +1,6 @@
 <?xml version="1.0"?>
 <robot xmlns:xacro="http://www.ros.org/wiki/xacro">
+<!--Camera description for the robot-->
+<!--Includes orientation, locations, various properties, and simulation instructions for Gazebo-->
     <joint name="camera_joint" type="fixed">
         <parent link="chassis"/>

File: description/contact_switch.xacro (robot description, xacro)
@@ -1,5 +1,8 @@
-<!--
+<!-- NOT SETUP OR USED YET
 <?xml version="1.0"?>
 <robot xmlns:xacro="http://www.ros.org/wiki/xacro">
+<!--Contact switch description for the robot-->
+<!--Includes orientation, locations, various properties, and simulation instructions for Gazebo-->
+<!--These are limit switches to sense when the robot touches an object, such as the charging dock-->
     <joint name="contact_joint" type="fixed">
         <parent link="chassis"/>

File: description/depth_camera.xacro (robot description, xacro)
@@ -1,4 +1,6 @@
 <?xml version="1.0"?>
 <robot xmlns:xacro="http://www.ros.org/wiki/xacro">
+<!--3D Depth Camera description for the robot-->
+<!--Includes orientation, locations, various properties, and simulation instructions for Gazebo-->
     <joint name="depth_camera_joint" type="fixed">
         <parent link="chassis"/>
@@ -23,12 +25,5 @@
         </xacro:inertial_box>
   </link>
-  <!--This rotates the camera image orientation to match
-  ROS coordinate standards
-    <joint name="depth_camera_optical_joint" type="fixed">
-        <origin xyz="0 0 0" rpy="${-pi/2} 0 ${-pi/2}" />
-        <parent link="depth_camera_link" />
-        <child link="depth_camera_link_optical" />
-    </joint>
-    <link name="depth_camera_link_optical"></link> -->
+<!-- Optical frame does not need to be rotated as it did for the rgb camera. I dont know why.-->
 <!--Gazebo plugin-->
     <gazebo reference="depth_camera_link">

File: description/imu.xacro (robot description, xacro)
@@ -1,4 +1,6 @@
 <?xml version="1.0"?>
 <robot xmlns:xacro="http://www.ros.org/wiki/xacro">
+<!--Inertial Measurement Unit sensor description for the robot-->
+<!--Includes orientation, locations, various properties, and simulation instructions for Gazebo-->
     <joint name="imu_joint" type="fixed">
         <parent link="chassis"/>

File: description/inertial_macros.xacro (robot description, xacro)
@@ -1,4 +1,5 @@
 <?xml version="1.0"?>
 <robot xmlns:xacro="http://www.ros.org/wiki/xacro" >
+    <!-- Macros to make physics calculations simpler -->
     <!-- Specify some standard inertial calculations https://en.wikipedia.org/wiki/List_of_moments_of_inertia -->
     <!-- These make use of xacro's mathematical functionality -->

File: description/lidar.xacro (robot description, xacro)
@@ -1,4 +1,6 @@
 <?xml version="1.0"?>
 <robot xmlns:xacro="http://www.ros.org/wiki/xacro" >
+<!--LIDAR description for the robot-->
+<!--Includes orientation, locations, various properties, and simulation instructions for Gazebo-->
     <!-- Lidar's urdf-->
     <joint name="laser_joint" type="fixed">

File: description/robot.urdf.xacro (robot description, xacro)
@@ -1,4 +1,6 @@
 <?xml version="1.0"?>
 <robot xmlns:xacro="http://www.ros.org/wiki/xacro"  name="robot">
+<!-- This is the main robot description file which pulls robot core, sensors, and control schemes together.-->
+ <!-- Everything could be here in one large file, but this approach is more organized and adaptable.-->
     <xacro:include filename="robot_core.xacro" /> <!--Base robot model-->
     <!-- <xacro:include filename="gazebo_control.xacro"/> -->

File: description/robot_core.xacro (robot description, xacro)
@@ -1,4 +1,5 @@
 <?xml version="1.0"?>
 <robot xmlns:xacro="http://www.ros.org/wiki/xacro">
+<!--This defines the physical structure and properties of the robot.-->
         <!-- Chassis Variables (all in metric) -->
     <xacro:property name="box_length" value="0.7"/> <!--meters-->

File: description/ros2_control.xacro (robot description, xacro)
@@ -1,4 +1,6 @@
 <?xml version="1.0"?>
 <robot xmlns:xacro="http://www.ros.org/wiki/xacro">
+<!--Adaptors to exchange info with Gazebo -->
+<!--Possibly same/same but different as gz_bridge.yaml method-->
     <ros2_control name="GazeboSystem" type="system">
         <hardware>
