Commit message: got my head striaghtened out, EKF smoother, back on track

File: description/depth_camera.xacro (robot description, xacro)
@@ -3,4 +3,5 @@
 <!--3D Depth Camera description for the robot-->
 <!--Includes orientation, locations, various properties, and simulation instructions for Gazebo-->
+<!--Reduced range(clip) from 15m to 7m, reduced framerate from 30Hz to 10Hz. This is for better performance and accuracy in simulation. -->
     <joint name="depth_camera_joint" type="fixed">
         <parent link="chassis"/>
@@ -56,15 +57,15 @@
                 <clip>
                     <near>0.1</near>
-                    <far>15</far>
+                    <far>7</far>
                 </clip>
                 <depth_camera>
                     <clip>
                         <near>0.1</near>
-                        <far>15</far>
+                        <far>7</far>
                     </clip>
                 </depth_camera>
             </camera>
             <always_on>1</always_on>
-            <update_rate>30</update_rate>
+            <update_rate>10</update_rate>
             <visualize>0</visualize>
             <topic>/depth_camera</topic>

File: description/imu.xacro (robot description, xacro)
@@ -8,88 +8,89 @@
         <origin xyz="0 0 0.15" rpy="0 0 0"/>
     </joint>
-<link name="imu_link">
-        <visual>
-            <geometry>
-              <box size="0.010 0.01 0.01"/>
-            </geometry>
-            <material name="red"/>
-        </visual>
-        <collision>
-          <geometry>
-              <box size="0.010 0.01 0.01"/>
-          </geometry>
-        </collision>
-        <xacro:inertial_box mass="0.1" x="0.01" y="0.01" z="0.01">
-            <origin xyz="0 0 0" rpy="0 0 0"/>
-        </xacro:inertial_box>
-  <sensor name="imu_sensor" type="imu">
-    <always_on>true</always_on>
-    <update_rate>100</update_rate>
-    <visualize>true</visualize>
-    <topic>imu</topic>
-    <gz_frame_id>imu_link</gz_frame_id>
-    <imu>
+  <link name="imu_link">
+    <visual>
+      <geometry>
+        <box size="0.010 0.01 0.01"/>
+      </geometry>
+      <material name="red"/>
+    </visual>
+    <collision>
+     <geometry>
+      <box size="0.010 0.01 0.01"/>
+     </geometry>
+    </collision>
+    <xacro:inertial_box mass="0.1" x="0.01" y="0.01" z="0.01">
+     <origin xyz="0 0 0" rpy="0 0 0"/>
+    </xacro:inertial_box>
+    <sensor name="imu_sensor" type="imu">
+     <always_on>true</always_on>
+     <update_rate>100</update_rate>
+     <visualize>true</visualize>
+     <topic>imu</topic>
+     <gz_frame_id>imu_link</gz_frame_id>
+     <imu>
       <angular_velocity>
-        <x>
-          <noise type="gaussian">
-            <mean>0.0</mean>
-            <stddev>2e-4</stddev>
-            <bias_mean>0.0000075</bias_mean>
-            <bias_stddev>0.0000008</bias_stddev>
-          </noise>
-        </x>
-        <y>
-          <noise type="gaussian">
-            <mean>0.0</mean>
-            <stddev>2e-4</stddev>
-            <bias_mean>0.0000075</bias_mean>
-            <bias_stddev>0.0000008</bias_stddev>
-          </noise>
-        </y>
-        <z>
-          <noise type="gaussian">
-            <mean>0.0</mean>
-            <stddev>2e-4</stddev>
-            <bias_mean>0.0000075</bias_mean>
-            <bias_stddev>0.0000008</bias_stddev>
-          </noise>
-        </z>
+      <x>
+        <noise type="gaussian">
+         <mean>0.0</mean>
+         <stddev>2e-4</stddev>
+         <bias_mean>0.0000075</bias_mean>
+         <bias_stddev>0.0000008</bias_stddev>
+        </noise>
+      </x>
+      <y>
+        <noise type="gaussian">
+         <mean>0.0</mean>
+         <stddev>2e-4</stddev>
+         <bias_mean>0.0000075</bias_mean>
+         <bias_stddev>0.0000008</bias_stddev>
+        </noise>
+      </y>
+       <z>
+        <noise type="gaussian">
+         <mean>0.0</mean>
+         <stddev>2e-4</stddev>
+         <bias_mean>0.0000075</bias_mean>
+         <bias_stddev>0.0000008</bias_stddev>
+        </noise>
+       </z>
       </angular_velocity>
       <linear_acceleration>
-        <x>
-          <noise type="gaussian">
-            <mean>0.0</mean>
-            <stddev>1.7e-2</stddev>
-            <bias_mean>0.1</bias_mean>
-            <bias_stddev>0.001</bias_stddev>
-          </noise>
-        </x>
-        <y>
-          <noise type="gaussian">
-            <mean>0.0</mean>
-            <stddev>1.7e-2</stddev>
-            <bias_mean>0.1</bias_mean>
-            <bias_stddev>0.001</bias_stddev>
-          </noise>
-        </y>
-        <z>
-          <noise type="gaussian">
-            <mean>0.0</mean>
-            <stddev>1.7e-2</stddev>
-            <bias_mean>0.1</bias_mean>
-            <bias_stddev>0.001</bias_stddev>
-          </noise>
-        </z>
+       <x>
+        <noise type="gaussian">
+         <mean>0.0</mean>
+         <stddev>1.7e-2</stddev>
+         <bias_mean>0.1</bias_mean>
+         <bias_stddev>0.001</bias_stddev>
+        </noise>
+       </x>
+       <y>
+        <noise type="gaussian">
+         <mean>0.0</mean>
+         <stddev>1.7e-2</stddev>
+         <bias_mean>0.1</bias_mean>
+         <bias_stddev>0.001</bias_stddev>
+        </noise>
+       </y>
+       <z>
+        <noise type="gaussian">
+         <mean>0.0</mean>
+         <stddev>1.7e-2</stddev>
+         <bias_mean>0.1</bias_mean>
+         <bias_stddev>0.001</bias_stddev>
+        </noise>
+       </z>
       </linear_acceleration>
-    </imu>
-  </sensor>
-</link>
+     </imu>
+    </sensor>
+  </link>
 <!--Gazebo plugin-->
     <gazebo reference="imu_link">
         <sensor name="imu_sensor" type="imu">
-            <always_on>1</always_on>
-            <update_rate>1</update_rate>
+          <always_on>1</always_on>
+          <update_rate>10</update_rate>
          <visualize>true</visualize>
-         <topic>imu</topic>
+         <topic>imu/data</topic>
+         <gz_frame_id>imu_link</gz_frame_id>
         </sensor>
     </gazebo>

File: description/robot.urdf.xacro (robot description, xacro)
@@ -8,5 +8,5 @@
     <xacro:include filename="lidar.xacro" />
     <xacro:include filename="camera.xacro" />
-    <xacro:include filename="depth_camera.xacro" />
+    <!-- <xacro:include filename="depth_camera.xacro" /> --> <!--Disabled depth camera for performance reasons-->
     <xacro:include filename="imu.xacro" />
     <!--<xacro:include filename="contact_switch.xacro" /> -->

File: description/robot_core.xacro (robot description, xacro)
@@ -2,15 +2,15 @@
 <robot xmlns:xacro="http://www.ros.org/wiki/xacro">
 <!--This defines the physical structure and properties of the robot.-->
-        <!-- Chassis Variables (all in metric) -->
-    <xacro:property name="box_length" value="0.7"/> <!--meters-->
+        <!-- Chassis Variables (all in meters/kg) -->
+    <xacro:property name="box_length" value="0.7"/> <!--Adjust footprint to reflect changes here-->
     <xacro:property name="box_width" value="0.35"/>
     <xacro:property name="box_height" value="0.15"/>
     <xacro:property name="box_mass" value="10"/>
-    <xacro:property name="wheel_width" value="0.075"/>
+    <xacro:property name="wheel_width" value="0.075"/> <!--Adjust footprint to reflect changes here-->
     <xacro:property name="wheel_radius" value="0.127"/>
     <xacro:property name="wheel_offset" value="${box_width/2 + wheel_width/2}"/>
     <xacro:property name="wheel_mass" value="1.0"/> <!--kg-->
     <xacro:property name="wheel_torque" value="50"/> <!--N.m-->
-    <xacro:property name="wheel_speed" value="10.0"/> <!--rad/s-->
+    <xacro:property name="wheel_speed" value="20.0"/> <!--rad/s-->
     <xacro:property name="caster_radius" value="0.0635"/>
     <xacro:property name="caster_Xoffset" value="${box_length - caster_radius}"/>

File: description/ros2_control.xacro (robot description, xacro)
@@ -2,6 +2,7 @@
 <robot xmlns:xacro="http://www.ros.org/wiki/xacro">
 <!--Adaptors to exchange info with Gazebo -->
-<!--Possibly same/same but different as gz_bridge.yaml method-->
-    <ros2_control name="GazeboSystem" type="system">
+<!--Possibly same/same but different as gz_bridge.yaml method?-->
+    <ros2_control name="GazeboSystem" type="system"> <!--For use with the simulator, as opposed to a physical bot-->
+     <!--https://beta.articulatedrobotics.xyz/tutorials/mobile-robot/applications/ros2_control-concepts-->
         <hardware>
             <plugin>gz_ros2_control/GazeboSimSystem</plugin>
@@ -24,5 +25,5 @@
         </joint>
     </ros2_control>
-    <gazebo>
+    <gazebo> <!--This is the second part of above, not a seperate idea-->
         <plugin name="gz_ros2_control::GazeboSimROS2ControlPlugin" filename="libgz_ros2_control-system.so">
             <!-- Make sure to put your package name in there!! -->
