Commit message: efk works now but /odom message has blank frame IDs still. Tuned up/changed lots of little things

File: description/imu.xacro (robot description, xacro)
@@ -4,7 +4,7 @@
 <!--Includes orientation, locations, various properties, and simulation instructions for Gazebo-->
     <joint name="imu_joint" type="fixed">
-        <parent link="chassis"/>
+        <parent link="base_link"/>
         <child link="imu_link"/>
-        <origin xyz="0 0 0.15" rpy="0 0 0"/>
+        <origin xyz="0.0 0.0 0.15" rpy="0 0 0"/>
     </joint>
   <link name="imu_link">
@@ -17,5 +17,5 @@
     <collision>
      <geometry>
-      <box size="0.010 0.01 0.01"/>
+      <box size="0.01 0.01 0.01"/>
      </geometry>
     </collision>
@@ -91,5 +91,5 @@
           <update_rate>10</update_rate>
          <visualize>true</visualize>
-         <topic>imu/data</topic>
+         <topic>/imu</topic>
          <gz_frame_id>imu_link</gz_frame_id>
         </sensor>

File: description/robot_core.xacro (robot description, xacro)
@@ -12,5 +12,5 @@
     <xacro:property name="wheel_mass" value="1.0"/> <!--kg-->
     <xacro:property name="wheel_torque" value="50"/> <!--N.m-->
-    <xacro:property name="wheel_speed" value="20.0"/> <!--rad/s-->
+    <xacro:property name="wheel_speed" value="5.0"/> <!--rad/s-->
     <xacro:property name="caster_radius" value="0.0635"/>
     <xacro:property name="caster_Xoffset" value="${box_length - caster_radius}"/>
