Commit message: added rear camera

File: description/rear_camera.xacro (robot description, xacro)
@@ -3,14 +3,14 @@
 <!--Camera description for the robot-->
 <!--Includes orientation, locations, various properties, and simulation instructions for Gazebo-->
-    <joint name="camera_joint" type="fixed">
+    <joint name="rear_camera_joint" type="fixed">
         <parent link="chassis"/>
-        <child link="camera_link"/>
-        <origin xyz="0.7005 0 0.1" rpy="0 0 0"/>
+        <child link="rear_camera_link"/>
+        <origin xyz="-0.01 0 0.1" rpy="0 0 ${pi/2}"/> <!--Faces backwards-->
     </joint>
     <!--This is the camera body in ROS coordinate standard-->
-    <link name="camera_link">
+    <link name="rear_camera_link">
         <visual>
             <geometry>
-              <box size="0.010 0.03 0.03"/>
+              <box size="0.01 0.03 0.03"/>
             </geometry>
             <material name="red"/>
@@ -27,18 +27,18 @@
   <!--This rotates the camera image orientation to match
   ROS coordinate standards-->
-    <joint name="camera_optical_joint" type="fixed">
+    <joint name="rear_camera_optical_joint" type="fixed">
         <origin xyz="0 0 0" rpy="${-pi/2} 0 ${-pi/2}" />
-        <parent link="camera_link" />
-        <child link="camera_link_optical" />
+        <parent link="rear_camera_link" />
+        <child link="rear_camera_link_optical" />
     </joint>
-    <link name="camera_link_optical"></link>
+    <link name="rear_camera_link_optical"></link>
 <!--Gazebo plugin-->
-    <gazebo reference="camera_link">
-        <sensor name="camera" type="camera">
-            <pose> 0 0 0 0 0 0 </pose>
+    <gazebo reference="rear_camera_link">
+        <sensor name="rear_camera" type="camera">
+            <pose> -0.01 0 0 0 0 ${pi/2} </pose> <!--Faces backwards-->
             <visualize>true</visualize>
             <update_rate>10</update_rate>
             <camera>
-                <camera_info_topic>camera/camera_info</camera_info_topic>
+                <camera_info_topic>rear_camera/camera_info</camera_info_topic>
                 <horizontal_fov>1.089</horizontal_fov>
                 <image>
@@ -52,6 +52,6 @@
                 </clip>
             </camera>
-            <topic>camera/image_raw</topic>
-            <gz_frame_id>camera_link_optical</gz_frame_id>
+            <topic>rear_camera/image_raw</topic>
+            <gz_frame_id>rear_camera_link_optical</gz_frame_id>
         </sensor>
     </gazebo>

File: description/robot.urdf.xacro (robot description, xacro)
@@ -7,5 +7,5 @@
     <xacro:include filename="ros2_control.xacro"/>
     <xacro:include filename="lidar.xacro" />
-    <xacro:include filename="camera.xacro" />
+    <xacro:include filename="rear_camera.xacro" />
     <!-- <xacro:include filename="depth_camera.xacro" /> --> <!--Disabled depth camera for performance reasons-->
     <xacro:include filename="imu.xacro" />
