Commit message: recovered launch, corrected cameras(maybe?)

File: description/garbo_description.urdf (robot description, URDF)
Before this commit: robot garbo, 7 links, 6 joints
Links:
- added link depth_camera_optical_link
- added link rear_camera_optical_link
Joints:
- added joint depth_camera_optical_joint: type fixed, parent depth_camera_link, child depth_camera_optical_link, origin xyz=0 0 0 rpy=${-pi/2} 0 ${-pi/2}
- added joint rear_camera_optical_joint: type fixed, parent rear_camera_link, child rear_camera_optical_link, origin xyz=0 0 0 rpy=${-pi/2} 0 ${-pi/2}
- joint depth_camera_joint: origin xyz=${base_length - wheel_radius + 0.005} 0 0.1 rpy=0 0 0 -> xyz=${base_length - wheel_radius + 0.005} 0 ${base_height - 0.015} rpy=0 0 0
- joint rear_camera_joint: origin xyz=${-wheel_radius-0.01} 0 0.1 rpy=0 0 ${pi} -> xyz=${-wheel_radius-0.01} 0 ${base_height - 0.015} rpy=0 0 ${-pi}

Commit message: apriltagTF on rear camera works; not yet on depth camera

File: description/garbo_description.urdf (robot description, URDF)
Before this commit: robot garbo, 9 links, 8 joints
Links:
- added link depth_camera_depth_link
Joints:
- added joint depth_camera_depth_joint: type fixed, parent depth_camera_link, child depth_camera_depth_link, origin xyz=0 0 0 rpy=0 0 0
- joint depth_camera_optical_joint: origin xyz=0 0 0 rpy=${-pi/2} 0 ${-pi/2} -> xyz=0 0 0 rpy=0 0 0

Commit message: depthcloud and TF aligned, PointCloud still misaligned but not needed for now

File: description/garbo_description.urdf (robot description, URDF)
Before this commit: robot garbo, 10 links, 9 joints
Links:
- removed link depth_camera_depth_link
- removed link rear_camera_link
- removed link rear_camera_optical_link
Joints:
- removed joint depth_camera_depth_joint
- removed joint rear_camera_joint
- removed joint rear_camera_optical_joint
- joint depth_camera_optical_joint: origin xyz=0 0 0 rpy=0 0 0 -> xyz=0 0 0 rpy=${-pi/2} 0 ${-pi/2}
